Commit message: finish: car model

File: src/turn_on_wheeltec_robot/urdf/senior_akm_robot.urdf (robot description, URDF)
Before this commit: robot wheeltec_robot, 5 links, 4 joints
Joints:
- joint left_front_joint: origin xyz=0.31 0.162 0.05 rpy=1.57 0 0 -> xyz=0.15 0.162 0.05 rpy=1.57 0 0
- joint left_wheel_joint: origin xyz=0 0.162 0.05 rpy=1.57 0 0 -> xyz=-0.15 0.162 0.05 rpy=1.57 0 0
- joint right_front_joint: origin xyz=0.31 -0.162 0.05 rpy=1.57 0 0 -> xyz=0.15 -0.162 0.05 rpy=1.57 0 0
- joint right_wheel_joint: origin xyz=0 -0.162 0.05 rpy=1.57 0 0 -> xyz=-0.15 -0.162 0.05 rpy=1.57 0 0
